Commit message: made the layout for the platform

File: src/printing_station/urdf/inspection_bot/robot.urdf (robot description, URDF)
Before this commit: robot simple_cylinder, 1 links, 0 joints
Links:
- link base_link: geometry collision cylinder length=1.8 radius=0.3; visual cylinder length=1.8 radius=0.11
