Commit message: second try of robot adding

File: src/URDF_Knickarmroboter/urdf/URDF_Knickarmroboter.urdf (robot description, URDF)
Before this commit: robot Knickarmroboter_URDF, 7 links, 6 joints
Links:
- link base_link: geometry collision mesh filename=package://URDF_Knickarmroboter/meshes/base_link.STL; visual mesh filename=package://URDF_Knickarmroboter/meshes/base_link.STL
- link l1: geometry collision mesh filename=package://URDF_Knickarmroboter/meshes/l1.STL; visual mesh filename=package://URDF_Knickarmroboter/meshes/l1.STL
- link l2: geometry collision mesh filename=package://URDF_Knickarmroboter/meshes/l2.STL; visual mesh filename=package://URDF_Knickarmroboter/meshes/l2.STL
- link l3: geometry collision mesh filename=package://URDF_Knickarmroboter/meshes/l3.STL; visual mesh filename=package://URDF_Knickarmroboter/meshes/l3.STL
- link l4: geometry collision mesh filename=package://URDF_Knickarmroboter/meshes/l4.STL; visual mesh filename=package://URDF_Knickarmroboter/meshes/l4.STL
- link l5: geometry collision mesh filename=package://URDF_Knickarmroboter/meshes/l5.STL; visual mesh filename=package://URDF_Knickarmroboter/meshes/l5.STL
- link l6: geometry collision mesh filename=package://URDF_Knickarmroboter/meshes/l6.STL; visual mesh filename=package://URDF_Knickarmroboter/meshes/l6.STL

Commit message: fixed roboter size

File: src/URDF_Knickarmroboter/urdf/URDF_Knickarmroboter.urdf (robot description, URDF)
Before this commit: robot URDF_Knickarmroboter, 7 links, 6 joints
Links:
- removed link l6
- link base_link: mass 1.98151152753041 -> 6.1361913950356
- link l1: mass 3.58989007226229 -> 1.51482515033566
- link l2: mass 2.15458853713248 -> 2.94963547245468
- link l3: mass 0.575994505699524 -> 0.478407770132196
- link l4: mass 1.0036372704856 -> 0.988047538826246
- link l5: mass 0.283355917359441 -> 0.280114187576556
Joints:
- removed joint j6
- joint j1: axis 0 0 1 -> 0 0 -1
- joint j2: axis -0.0066494 0.99998 0 -> 0.062633 -0.99804 0
- joint j3: axis -0.0066494 0.99998 0 -> -0.062633 0.99804 0
- joint j4: axis -0.99986 -0.0066486 0.01561 -> -0.99804 -0.062633 0
- joint j5: axis -0.007173 0.9994 -0.033783 -> -0.062633 0.99804 0

File: src/printing_station/urdf/printer_stand.urdf (robot description, URDF)
Before this commit: robot simple_box, 1 links, 0 joints
Links:
- link base_link: geometry collision box size=0.8 0.3 0.4; visual box size=0.8 0.3 0.4
