Commit message: added full station but with a weird 4 axis

File: src/fertig/urdf/fertig.urdf (robot description, URDF)
Before this commit: robot full_station, 13 links, 12 joints
Links:
- removed link drucker
- added link knick_link5, mass 0.31824; collision mesh filename=package://fertig/meshes/knick_link5.STL; visual mesh filename=package://fertig/meshes/knick_link5.STL
- added link knick_link6, mass 0.226630428770624; collision mesh filename=package://fertig/meshes/knick_link6.STL; visual mesh filename=package://fertig/meshes/knick_link6.STL
- added link tisch, mass 0; collision mesh filename=package://fertig/meshes/tisch.STL; visual mesh filename=package://fertig/meshes/tisch.STL
- link boxes: geometry collision mesh filename=package://fertig/meshes/boxes.STL; visual mesh filename=package://fertig/meshes/boxes.STL
- link knick_base_link: geometry collision mesh filename=package://fertig/meshes/knick_base_link.STL; visual mesh filename=package://fertig/meshes/knick_base_link.STL
- link knick_link1: geometry collision mesh filename=package://fertig/meshes/knick_link1.STL; visual mesh filename=package://fertig/meshes/knick_link1.STL
- link knick_link2: mass 2.94963527631575 -> 2.94963721988334; geometry collision mesh filename=package://fertig/meshes/knick_link2.STL; visual mesh filename=package://fertig/meshes/knick_link2.STL
- link knick_link3: mass 0.491452048874692 -> 0.491452097756812; geometry collision mesh filename=package://fertig/meshes/knick_link3.STL; visual mesh filename=package://fertig/meshes/knick_link3.STL
- link knick_link4: mass 0.988047540426667 -> 0.98805; geometry collision mesh filename=package://fertig/meshes/knick_link4.STL; visual mesh filename=package://fertig/meshes/knick_link4.STL
- link knickarm_sockel: geometry collision mesh filename=package://fertig/meshes/knickarm_sockel.STL; visual mesh filename=package://fertig/meshes/knickarm_sockel.STL
- link scara_link_1: geometry collision mesh filename=package://fertig/meshes/scara_link_1.STL; visual mesh filename=package://fertig/meshes/scara_link_1.STL
- link scara_link_2: geometry collision mesh filename=package://fertig/meshes/scara_link_2.STL; visual mesh filename=package://fertig/meshes/scara_link_2.STL
- link scara_link_3: geometry collision mesh filename=package://fertig/meshes/scara_link_3.STL; visual mesh filename=package://fertig/meshes/scara_link_3.STL
- link scara_link_base: geometry collision mesh filename=package://fertig/meshes/scara_link_base.STL; visual mesh filename=package://fertig/meshes/scara_link_base.STL
- link world_link: geometry collision mesh filename=package://fertig/meshes/world_link.STL; visual mesh filename=package://fertig/meshes/world_link.STL
Joints:
- removed joint drucker
- added joint knick_joint5: type revolute, parent knick_link4, child knick_link5, origin xyz=0.035397 0.01714 0.185 rpy=1.5708 -1.0202 -1.1491, axis 0 0 1, limit lower=-3 upper=3 effort=0 velocity=0
- added joint knick_joint6: type revolute, parent knick_link5, child knick_link6, origin xyz=0.07015 0.10346 0.039 rpy=-1.5708 0.97279 -0.59583, axis 0 0 1, limit lower=3 upper=3 effort=0 velocity=0
- added joint tisch: type fixed, parent world_link, child tisch, origin xyz=-1.07 2.523 -0.0199999999999989 rpy=1.5707963267949 -1.5707963267949 0, axis 0 0 0
- joint knick_joint3: origin xyz=-0.001388 0.3 0.02 rpy=0 0 0 -> xyz=-0.051008 0.29563 0.02 rpy=0 0 0
- joint knick_joint4: origin xyz=0.15497 -0.0031424 0.052879 rpy=-0.14998 1.5708 -0.16421 -> xyz=0.13566 0.074989 0.052879 rpy=0.5106 1.5708 0
- joint scara_joint_1: limit lower=-3 upper=3 effort=0 velocity=0 -> lower=-2.5 upper=2.5 effort=0 velocity=0; origin xyz=0 0.0620000000000001 0.185999999999999 rpy=0 0 0 -> xyz=0 0.062 0.186 rpy=0 0 0
- joint scara_joint_2: limit lower=-3 upper=3 effort=0 velocity=0 -> lower=-2.5 upper=2.5 effort=0 velocity=0; origin xyz=0.110915088922781 0.331544853874781 0.0550000000000013 rpy=0 0 0 -> xyz=0.11092 0.33154 0.055 rpy=0 0 0
- joint scara_joint_3: limit lower=-0.25 upper=0 effort=0 velocity=0 -> lower=-2.5 upper=2.5 effort=0 velocity=0; origin xyz=0.217106821845328 0.394163199586445 0 rpy=3.14159265358979 0 -3.14159265358979 -> xyz=0.21711 0.39416 0 rpy=3.1416 0 -3.1416
