Commit message: runs now

File: src/gesamt_station/urdf/gesamt_station.urdf (robot description, URDF)
Before this commit: robot gesamt_station, 15 links, 14 joints
Joints:
- joint knick_joint1: limit lower=-3 upper=3 effort=0 velocity=0 -> lower=-3 upper=3 effort=1000 velocity=20
- joint knick_joint2: limit lower=-3 upper=3 effort=0 velocity=0 -> lower=-3 upper=3 effort=1000 velocity=20
- joint knick_joint3: limit lower=-3 upper=3 effort=0 velocity=0 -> lower=-3 upper=3 effort=1000 velocity=20
- joint knick_joint4: limit lower=-3 upper=3 effort=0 velocity=0 -> lower=-3 upper=3 effort=1000 velocity=20
- joint knick_joint5: limit lower=-3 upper=3 effort=0 velocity=0 -> lower=-3 upper=3 effort=1000 velocity=20
- joint knick_joint6: limit lower=-3 upper=3 effort=0 velocity=0 -> lower=-3 upper=3 effort=1000 velocity=20
- joint scara_joint_1: limit lower=-2.5 upper=2.5 effort=0 velocity=0 -> lower=-2.5 upper=2.5 effort=1000 velocity=20
- joint scara_joint_2: limit lower=-2.5 upper=2.5 effort=0 velocity=0 -> lower=-2.5 upper=2.5 effort=1000 velocity=20
- joint scara_joint_3: limit lower=-2.5 upper=2.5 effort=0 velocity=0 -> lower=-2.5 upper=2.5 effort=1000 velocity=20

Commit message: cleaned the workspace, added python script to send goal poses

File: src/gesamt_station/urdf/gesamt_station.urdf (robot description, URDF)
Before this commit: robot gesamt_station, 15 links, 14 joints
Joints:
- joint scara_joint_3: limit lower=-2.5 upper=2.5 effort=1000 velocity=20 -> lower=-0.2 upper=0.2 effort=1000 velocity=20
